Commit message: feat: add robot_vision_tools and manage easy_handeye2 as submodule (https://github.com/marcoesposito1988/easy_handeye2)

File: src/integrated_robot/robot_description/urdf/integrated_robot.urdf.xacro (robot description, xacro)
@@ -95,5 +95,5 @@
       <!-- Camera attached to tool_link -->
       <xacro:realsense_camera parent="tool_link">
-        <origin xyz="-0.049074 0.048515 0.06645" rpy="0.066568 0 -2.3363"/>
+        <origin xyz="-0.013298 0.067929 0.041207" rpy="-0.001305 -0.024822 -2.612690"/>
       </xacro:realsense_camera>
     </xacro:if>
